File: engineering/electronics/pcbs/BMSJ/kicad/BMSJ.kicad_pcb (KiCad board)
At the start: 2 copper layers, 0 parts

Commit message: Kicad_Update
- Add busbar cell connection
- Screw holes
- Edge cuts
Routing:
- added copper zone on F.Cu, net (none)
Other:
- board outline added: 200 x 115 mm

Commit message: KiCad_Update
Parts:
- added C1: 100p, Capacitor_SMD:C_0603_1608Metric, F.Cu at (1.50, 0.76)
- added C10: 1u, Capacitor_SMD:C_0805_2012Metric, F.Cu at (46.5, 26.0)
- added C11: 100n, Capacitor_SMD:C_0603_1608Metric, F.Cu at (1.50, 10.8)
- added C12: 100n, Capacitor_SMD:C_0603_1608Metric, F.Cu at (1.50, 13.3)
- added C13: 100n, Capacitor_SMD:C_0603_1608Metric, F.Cu at (1.50, 15.8)
- added C14: 100n, Capacitor_SMD:C_0603_1608Metric, F.Cu at (1.50, 18.3)
- added C15: 100n, Capacitor_SMD:C_0603_1608Metric, F.Cu at (1.50, 20.8)
- added C16: 100n, Capacitor_SMD:C_0603_1608Metric, F.Cu at (1.50, 23.3)
- added C17: 100n, Capacitor_SMD:C_0603_1608Metric, F.Cu at (1.50, 25.9)
- added C18: 100n, Capacitor_SMD:C_0603_1608Metric, F.Cu at (1.50, 28.4)
- added C19: 100n, Capacitor_SMD:C_0603_1608Metric, F.Cu at (1.50, 30.9)
- added C2: 100p, Capacitor_SMD:C_0603_1608Metric, F.Cu at (1.50, 3.27)
- added C20: 100n, Capacitor_SMD:C_0603_1608Metric, F.Cu at (5.51, 0.76)
- added C21: 100p, Capacitor_SMD:C_0603_1608Metric, F.Cu at (5.51, 3.27)
- added C22: 100p, Capacitor_SMD:C_0603_1608Metric, F.Cu at (5.51, 5.78)
- added C23: 22u, Capacitor_SMD:C_0805_2012Metric, F.Cu at (46.5, 29.0)
- added C24: 22u, Capacitor_SMD:C_0805_2012Metric, F.Cu at (46.5, 32.0)
- added C25: 100n, Capacitor_SMD:C_0603_1608Metric, F.Cu at (5.51, 8.29)
- added C26: 100n, Capacitor_SMD:C_0603_1608Metric, F.Cu at (5.51, 10.8)
- added C27: 1u, Capacitor_SMD:C_0805_2012Metric, F.Cu at (46.5, 35.0)
- added C28: 47n, Capacitor_SMD:C_0603_1608Metric, F.Cu at (5.51, 13.3)
- added C29: 10u, Capacitor_SMD:C_0603_1608Metric, F.Cu at (5.51, 15.8)
- added C3: 100n, Capacitor_SMD:C_0603_1608Metric, F.Cu at (1.50, 5.78)
- added C30: 10u, Capacitor_SMD:C_0603_1608Metric, F.Cu at (5.51, 18.3)
- added C31: 10u, Capacitor_SMD:C_0603_1608Metric, F.Cu at (5.51, 20.8)
- added C32: 1u, Capacitor_SMD:C_0805_2012Metric, F.Cu at (46.5, 38.0)
- added C33: 1u, Capacitor_SMD:C_0805_2012Metric, F.Cu at (50.9, 26.0)
- added C34: 1u, Capacitor_SMD:C_0805_2012Metric, F.Cu at (50.9, 29.0)
- added C35: 1u, Capacitor_SMD:C_0805_2012Metric, F.Cu at (50.9, 32.0)
- added C36: 1u, Capacitor_SMD:C_0805_2012Metric, F.Cu at (50.9, 35.0)
- added C37: 2.2u, Capacitor_SMD:C_0603_1608Metric, F.Cu at (5.51, 23.3)
- added C38: 100n, Capacitor_SMD:C_0603_1608Metric, F.Cu at (5.51, 25.9)
- added C39: 100n, Capacitor_SMD:C_0603_1608Metric, F.Cu at (5.51, 28.4)
- added C4: 100n, Capacitor_SMD:C_0603_1608Metric, F.Cu at (1.50, 8.29)
- added C40: 100n, Capacitor_SMD:C_0603_1608Metric, F.Cu at (5.51, 30.9)
- added C41: 100n, Capacitor_SMD:C_0603_1608Metric, F.Cu at (9.53, 0.76)
- added C42: 100n, Capacitor_SMD:C_0603_1608Metric, F.Cu at (9.53, 3.27)
- added C43: 100n, Capacitor_SMD:C_0603_1608Metric, F.Cu at (56.1, 91.3)
- added C44: 100n, Capacitor_SMD:C_0603_1608Metric, F.Cu at (34.3, 62.4)
- added C45: 100n, Capacitor_SMD:C_0603_1608Metric, F.Cu at (77.9, 76.9)
- added C46: 100n, Capacitor_SMD:C_0603_1608Metric, F.Cu at (23.3, 62.4)
- added C47: 100n, Capacitor_SMD:C_0603_1608Metric, F.Cu at (69.0, 34.7)
- added C48: 100n, Capacitor_SMD:C_0603_1608Metric, F.Cu at (67.0, 62.4)
- added C49: 100n, Capacitor_SMD:C_0603_1608Metric, F.Cu at (67.0, 76.9)
- added C5: 1u, Capacitor_SMD:C_0805_2012Metric, F.Cu at (42.0, 26.0)
- added C50: 100n, Capacitor_SMD:C_0603_1608Metric, F.Cu at (12.4, 76.9)
- added C51: 100n, Capacitor_SMD:C_0603_1608Metric, F.Cu at (12.4, 62.4)
- added C52: 100n, Capacitor_SMD:C_0603_1608Metric, F.Cu at (45.2, 91.3)
- added C53: 100n, Capacitor_SMD:C_0603_1608Metric, F.Cu at (12.4, 91.3)
- added C54: 100n, Capacitor_SMD:C_0603_1608Metric, F.Cu at (1.50, 76.9)
- added C55: 100n, Capacitor_SMD:C_0603_1608Metric, F.Cu at (23.3, 76.9)
- added C56: 100n, Capacitor_SMD:C_0603_1608Metric, F.Cu at (1.50, 91.3)
- added C57: 100n, Capacitor_SMD:C_0603_1608Metric, F.Cu at (56.1, 62.4)
- added C58: 100n, Capacitor_SMD:C_0603_1608Metric, F.Cu at (45.2, 76.9)
- added C59: 100n, Capacitor_SMD:C_0603_1608Metric, F.Cu at (34.3, 91.3)
- added C6: 1u, Capacitor_SMD:C_0805_2012Metric, F.Cu at (42.0, 29.0)
- added C60: 100n, Capacitor_SMD:C_0603_1608Metric, F.Cu at (77.9, 62.4)
- added C61: 100n, Capacitor_SMD:C_0603_1608Metric, F.Cu at (58.1, 34.7)
- added C62: 100n, Capacitor_SMD:C_0603_1608Metric, F.Cu at (56.1, 76.9)
- added C63: 100n, Capacitor_SMD:C_0603_1608Metric, F.Cu at (34.3, 76.9)
- added C64: 100n, Capacitor_SMD:C_0603_1608Metric, F.Cu at (1.50, 62.4)
- added C65: 100n, Capacitor_SMD:C_0603_1608Metric, F.Cu at (45.2, 62.4)
- added C66: 100n, Capacitor_SMD:C_0603_1608Metric, F.Cu at (23.3, 91.3)
- added C67: 10n, Capacitor_SMD:C_0603_1608Metric, F.Cu at (58.1, 0.76)
- added C68: 10n, Capacitor_SMD:C_0603_1608Metric, F.Cu at (58.1, 3.27)
- added C69: 1u, Capacitor_SMD:C_0603_1608Metric, F.Cu at (58.1, 5.78)
- added C7: 1u, Capacitor_SMD:C_0805_2012Metric, F.Cu at (42.0, 32.0)
- added C70: 100n, Capacitor_SMD:C_0603_1608Metric, F.Cu at (58.1, 8.29)
- added C71: 1u, Capacitor_SMD:C_0805_2012Metric, F.Cu at (74.4, 6.32)
- added C72: 100n, Capacitor_SMD:C_0603_1608Metric, F.Cu at (58.1, 10.8)
- added C73: 1u, Capacitor_SMD:C_0805_2012Metric, F.Cu at (74.4, 9.32)
- added C74: 100n, Capacitor_SMD:C_0603_1608Metric, F.Cu at (58.1, 13.3)
- added C75: 10n, Capacitor_SMD:C_0805_2012Metric, F.Cu at (74.4, 12.3)
- added C76: 100n, Capacitor_SMD:C_0603_1608Metric, F.Cu at (58.1, 15.8)
- added C77: 18p, Capacitor_SMD:C_0603_1608Metric, F.Cu at (58.1, 18.3)
- added C78: 18p, Capacitor_SMD:C_0603_1608Metric, F.Cu at (62.1, 0.76)
- added C79: 100n, Capacitor_SMD:C_0603_1608Metric, F.Cu at (62.1, 3.27)
- added C8: 1u, Capacitor_SMD:C_0805_2012Metric, F.Cu at (42.0, 35.0)
- added C80: 100n, Capacitor_SMD:C_0603_1608Metric, F.Cu at (62.1, 5.78)
- added C81: 2.2u, Capacitor_SMD:C_0603_1608Metric, F.Cu at (62.1, 8.29)
- added C82: 2.2u, Capacitor_SMD:C_0603_1608Metric, F.Cu at (62.1, 10.8)
- added C83: 2.2u, Capacitor_SMD:C_0603_1608Metric, F.Cu at (62.1, 13.3)
- added C9: 1u, Capacitor_SMD:C_0805_2012Metric, F.Cu at (42.0, 38.0)
- added D1: 1N4148W, Diode_SMD:D_SOD-123, F.Cu at (51.2, 1.18)
- added D10: BZT52H-C62, Diode_SMD:D_SOD-123, F.Cu at (51.2, 17.9)
- added D17: LED, LED_SMD:LED_0603_1608Metric, F.Cu at (50.6, 43.4)
- added D19: POWER, LED_SMD:LED_0603_1608Metric, F.Cu at (50.6, 46.0)
- added D2: 1N4148W, Diode_SMD:D_SOD-123, F.Cu at (51.2, 4.53)
- added D20: STATUS, LED_SMD:LED_0603_1608Metric, F.Cu at (50.6, 48.6)
- added D21: PDZ7.5B, Diode_SMD:D_SOD-323, F.Cu at (60.3, 96.0)
- added D22: PDZ7.5B, Diode_SMD:D_SOD-323, F.Cu at (38.4, 67.1)
- added D23: PDZ7.5B, Diode_SMD:D_SOD-323, F.Cu at (82.1, 81.5)
- added D24: PDZ7.5B, Diode_SMD:D_SOD-323, F.Cu at (27.5, 67.1)
- added D25: PDZ7.5B, Diode_SMD:D_SOD-323, F.Cu at (73.2, 39.4)
- added D26: PDZ7.5B, Diode_SMD:D_SOD-323, F.Cu at (71.2, 67.1)
- added D27: PDZ7.5B, Diode_SMD:D_SOD-323, F.Cu at (71.2, 81.5)
- added D28: PDZ7.5B, Diode_SMD:D_SOD-323, F.Cu at (16.6, 81.5)
- added D29: PDZ7.5B, Diode_SMD:D_SOD-323, F.Cu at (16.6, 67.1)
- added D3: BZT52H-C62, Diode_SMD:D_SOD-123, F.Cu at (51.2, 7.88)
- added D30: PDZ7.5B, Diode_SMD:D_SOD-323, F.Cu at (49.4, 96.0)
- added D31: PDZ7.5B, Diode_SMD:D_SOD-323, F.Cu at (16.6, 96.0)
- added D32: PDZ7.5B, Diode_SMD:D_SOD-323, F.Cu at (5.68, 81.5)
- added D33: PDZ7.5B, Diode_SMD:D_SOD-323, F.Cu at (27.5, 81.5)
- added D34: PDZ7.5B, Diode_SMD:D_SOD-323, F.Cu at (5.68, 96.0)
- added D35: PDZ7.5B, Diode_SMD:D_SOD-323, F.Cu at (60.3, 67.1)
- added D36: PDZ7.5B, Diode_SMD:D_SOD-323, F.Cu at (49.4, 81.5)
- added D37: PDZ7.5B, Diode_SMD:D_SOD-323, F.Cu at (38.4, 96.0)
- added D38: PDZ7.5B, Diode_SMD:D_SOD-323, F.Cu at (82.1, 67.1)
- added D39: PDZ7.5B, Diode_SMD:D_SOD-323, F.Cu at (62.3, 39.4)
- added D4: smcj150a, Diode_SMD:D_SMC, F.Cu at (42.9, 3.38)
- added D40: PDZ7.5B, Diode_SMD:D_SOD-323, F.Cu at (60.3, 81.5)
- added D41: PDZ7.5B, Diode_SMD:D_SOD-323, F.Cu at (38.4, 81.5)
- added D42: PDZ7.5B, Diode_SMD:D_SOD-323, F.Cu at (5.68, 67.1)
- added D43: PDZ7.5B, Diode_SMD:D_SOD-323, F.Cu at (49.4, 67.1)
- added D44: PDZ7.5B, Diode_SMD:D_SOD-323, F.Cu at (27.5, 96.0)
- added D5: smcj150a, Diode_SMD:D_SMC, F.Cu at (42.9, 11.1)
- added D6: smcj150a, Diode_SMD:D_SMC, F.Cu at (42.9, 18.9)
- added D7: LED, LED_SMD:LED_0603_1608Metric, F.Cu at (50.6, 40.8)
- added D8: 1N4148W, Diode_SMD:D_SOD-123, F.Cu at (51.2, 11.2)
- added D9: 1N4148W, Diode_SMD:D_SOD-123, F.Cu at (51.2, 14.6)
- added FB1: 33, Resistor_SMD:R_0603_1608Metric, F.Cu at (9.53, 5.78)
- added FB2: 33, Resistor_SMD:R_0603_1608Metric, F.Cu at (9.53, 8.29)
- added J1: - Power +, Connector_Phoenix_MC_HighVoltage:PhoenixContact_MCV_1,5_2-G-5.08_1x02_P5.08mm_Vertical, F.Cu at (31.2, 29.9)
- added J17: Temp, Connector_PinHeader_2.54mm:PinHeader_1x05_P2.54mm_Horizontal, F.Cu at (1.79, 34.4)
- added J19: Charger +, Connector_Phoenix_MC_HighVoltage:PhoenixContact_MCV_1,5_2-G-5.08_1x02_P5.08mm_Vertical, F.Cu at (31.2, 39.2)
- added J32: Temp, Connector_PinHeader_2.54mm:PinHeader_1x05_P2.54mm_Horizontal, F.Cu at (15.2, 34.4)
- added J35: ET60S-D06-0-00-D06-X-V1-S, BMSJ:SAMTEC_ET60S-D06-0-00-D06-X-V1-S, F.Cu at (200.2, 117.6)
- added J37: DEBUG, Connector_Molex:Molex_PicoBlade_53398-0571_1x05-1MP_P1.25mm_Vertical, F.Cu at (63.2, 22.5)
- added J38: USB, Connector_USB:USB_Micro-B_Molex-105133-0001, F.Cu at (77.2, 2.15)
- added Q1: IRFL4105PBF, Package_TO_SOT_SMD:SOT-223, F.Cu at (32.5, 3.70)
- added Q11: DMG2305UX-7, Package_TO_SOT_SMD:SOT-23, F.Cu at (60.6, 92.3)
- added Q12: DMG2305UX-7, Package_TO_SOT_SMD:SOT-23, F.Cu at (38.7, 63.4)
- added Q13: DMG2305UX-7, Package_TO_SOT_SMD:SOT-23, F.Cu at (82.4, 77.8)
- added Q14: DMG2305UX-7, Package_TO_SOT_SMD:SOT-23, F.Cu at (27.8, 63.4)
- added Q15: DMG2305UX-7, Package_TO_SOT_SMD:SOT-23, F.Cu at (73.5, 35.7)
- added Q16: DMG2305UX-7, Package_TO_SOT_SMD:SOT-23, F.Cu at (71.5, 63.4)
- added Q17: DMG2305UX-7, Package_TO_SOT_SMD:SOT-23, F.Cu at (71.5, 77.8)
- added Q18: DMG2305UX-7, Package_TO_SOT_SMD:SOT-23, F.Cu at (16.9, 77.8)
- added Q19: DMG2305UX-7, Package_TO_SOT_SMD:SOT-23, F.Cu at (16.9, 63.4)
- added Q20: DMG2305UX-7, Package_TO_SOT_SMD:SOT-23, F.Cu at (49.6, 92.3)
- added Q21: DMG2305UX-7, Package_TO_SOT_SMD:SOT-23, F.Cu at (16.9, 92.3)
- added Q22: DMG2305UX-7, Package_TO_SOT_SMD:SOT-23, F.Cu at (5.96, 77.8)
- added Q23: DMG2305UX-7, Package_TO_SOT_SMD:SOT-23, F.Cu at (27.8, 77.8)
- added Q24: DMG2305UX-7, Package_TO_SOT_SMD:SOT-23, F.Cu at (5.96, 92.3)
- added Q25: DMG2305UX-7, Package_TO_SOT_SMD:SOT-23, F.Cu at (60.6, 63.4)
- added Q26: DMG2305UX-7, Package_TO_SOT_SMD:SOT-23, F.Cu at (49.6, 77.8)
- added Q27: DMG2305UX-7, Package_TO_SOT_SMD:SOT-23, F.Cu at (38.7, 92.3)
- added Q28: DMG2305UX-7, Package_TO_SOT_SMD:SOT-23, F.Cu at (82.4, 63.4)
- added Q29: DMG2305UX-7, Package_TO_SOT_SMD:SOT-23, F.Cu at (62.6, 35.7)
- added Q3: IRFL4105PBF, Package_TO_SOT_SMD:SOT-223, F.Cu at (32.5, 12.0)
- added Q30: DMG2305UX-7, Package_TO_SOT_SMD:SOT-23, F.Cu at (60.6, 77.8)
- added Q31: DMG2305UX-7, Package_TO_SOT_SMD:SOT-23, F.Cu at (38.7, 77.8)
- added Q32: DMG2305UX-7, Package_TO_SOT_SMD:SOT-23, F.Cu at (5.96, 63.4)
- added Q33: DMG2305UX-7, Package_TO_SOT_SMD:SOT-23, F.Cu at (49.6, 63.4)
- added Q34: DMG2305UX-7, Package_TO_SOT_SMD:SOT-23, F.Cu at (27.8, 92.3)
- added Q4: IRFL4105PBF, Package_TO_SOT_SMD:SOT-223, F.Cu at (32.5, 20.4)
- added R1: 100, Resistor_SMD:R_0603_1608Metric, F.Cu at (9.53, 10.8)
- added R10: 0, Resistor_SMD:R_0603_1608Metric, F.Cu at (9.53, 30.9)
- added R100: 1.2k, Resistor_SMD:R_0603_1608Metric, F.Cu at (1.50, 81.9)
- added R101: 3.9, Resistor_SMD:R_2512_6332Metric, F.Cu at (3.85, 73.1)
- added R102: 100, Resistor_SMD:R_0603_1608Metric, F.Cu at (23.3, 79.4)
- added R103: 1.2k, Resistor_SMD:R_0603_1608Metric, F.Cu at (23.3, 81.9)
- added R104: 3.9, Resistor_SMD:R_2512_6332Metric, F.Cu at (25.7, 73.1)
- added R105: 100, Resistor_SMD:R_0603_1608Metric, F.Cu at (1.50, 93.8)
- added R106: 1.2k, Resistor_SMD:R_0603_1608Metric, F.Cu at (1.50, 96.3)
- added R107: 3.9, Resistor_SMD:R_2512_6332Metric, F.Cu at (3.85, 87.6)
- added R108: 100, Resistor_SMD:R_0603_1608Metric, F.Cu at (56.1, 64.9)
- added R109: 1.2k, Resistor_SMD:R_0603_1608Metric, F.Cu at (56.1, 67.4)
- added R11: 1M, Resistor_SMD:R_0603_1608Metric, F.Cu at (13.5, 0.76)
- added R110: 3.9, Resistor_SMD:R_2512_6332Metric, F.Cu at (58.5, 58.7)
- added R111: 100, Resistor_SMD:R_0603_1608Metric, F.Cu at (45.2, 79.4)
- added R112: 1.2k, Resistor_SMD:R_0603_1608Metric, F.Cu at (45.2, 81.9)
- added R113: 3.9, Resistor_SMD:R_2512_6332Metric, F.Cu at (47.5, 73.1)
- added R114: 100, Resistor_SMD:R_0603_1608Metric, F.Cu at (34.3, 93.8)
- added R115: 1.2k, Resistor_SMD:R_0603_1608Metric, F.Cu at (34.3, 96.3)
- added R116: 3.9, Resistor_SMD:R_2512_6332Metric, F.Cu at (36.6, 87.6)
- added R117: 100, Resistor_SMD:R_0603_1608Metric, F.Cu at (77.9, 64.9)
- added R118: 1.2k, Resistor_SMD:R_0603_1608Metric, F.Cu at (77.9, 67.4)
- added R119: 3.9, Resistor_SMD:R_2512_6332Metric, F.Cu at (80.3, 58.7)
- added R12: 0, Resistor_SMD:R_0603_1608Metric, F.Cu at (13.5, 3.27)
- added R120: 100, Resistor_SMD:R_0603_1608Metric, F.Cu at (58.1, 37.2)
- added R121: 1.2k, Resistor_SMD:R_0603_1608Metric, F.Cu at (58.1, 39.7)
- added R122: 3.9, Resistor_SMD:R_2512_6332Metric, F.Cu at (60.5, 31.0)
- added R123: 100, Resistor_SMD:R_0603_1608Metric, F.Cu at (56.1, 79.4)
- added R124: 1.2k, Resistor_SMD:R_0603_1608Metric, F.Cu at (56.1, 81.9)
- added R125: 3.9, Resistor_SMD:R_2512_6332Metric, F.Cu at (58.5, 73.1)
- added R126: 100, Resistor_SMD:R_0603_1608Metric, F.Cu at (34.3, 79.4)
- added R127: 1.2k, Resistor_SMD:R_0603_1608Metric, F.Cu at (34.3, 81.9)
- added R128: 3.9, Resistor_SMD:R_2512_6332Metric, F.Cu at (36.6, 73.1)
- added R129: 100, Resistor_SMD:R_0603_1608Metric, F.Cu at (1.50, 64.9)
- added R13: 10, Resistor_SMD:R_0603_1608Metric, F.Cu at (13.5, 5.78)
- added R130: 1.2k, Resistor_SMD:R_0603_1608Metric, F.Cu at (1.50, 67.4)
- added R131: 3.9, Resistor_SMD:R_2512_6332Metric, F.Cu at (3.85, 58.7)
- added R132: 100, Resistor_SMD:R_0603_1608Metric, F.Cu at (45.2, 64.9)
- added R133: 1.2k, Resistor_SMD:R_0603_1608Metric, F.Cu at (45.2, 67.4)
- added R134: 3.9, Resistor_SMD:R_2512_6332Metric, F.Cu at (47.5, 58.7)
- added R135: 100, Resistor_SMD:R_0603_1608Metric, F.Cu at (23.3, 93.8)
- added R136: 1.2k, Resistor_SMD:R_0603_1608Metric, F.Cu at (23.3, 96.3)
- added R137: 3.9, Resistor_SMD:R_2512_6332Metric, F.Cu at (25.7, 87.6)
- added R138: 51, Resistor_SMD:R_0603_1608Metric, F.Cu at (62.1, 15.8)
- added R139: 51, Resistor_SMD:R_0603_1608Metric, F.Cu at (62.1, 18.3)
- added R14: 4.7M, Resistor_SMD:R_0603_1608Metric, F.Cu at (13.5, 8.29)
- added R140: 806, Resistor_SMD:R_0603_1608Metric, F.Cu at (66.1, 0.76)
- added R141: 1.2k, Resistor_SMD:R_0603_1608Metric, F.Cu at (66.1, 3.27)
- added R142: 2.2k, Resistor_SMD:R_0603_1608Metric, F.Cu at (66.1, 5.78)
- added R143: 4.7M, Resistor_SMD:R_0805_2012Metric, F.Cu at (78.8, 6.29)
- added R144: 100k, Resistor_SMD:R_0603_1608Metric, F.Cu at (66.1, 8.29)
- added R145: 2.2k, Resistor_SMD:R_0603_1608Metric, F.Cu at (66.1, 10.8)
- added R146: 10k, Resistor_SMD:R_0603_1608Metric, F.Cu at (66.1, 13.3)
- added R147: 10k, Resistor_SMD:R_0603_1608Metric, F.Cu at (66.1, 15.8)
- added R148: 4.75k, Resistor_SMD:R_0603_1608Metric, F.Cu at (66.1, 18.3)
- added R149: 4.75k, Resistor_SMD:R_0603_1608Metric, F.Cu at (70.1, 0.76)
- added R15: 100k, Resistor_SMD:R_0603_1608Metric, F.Cu at (13.5, 10.8)
- added R150: 240, Resistor_SMD:R_0603_1608Metric, F.Cu at (70.1, 3.27)
- added R151: 240, Resistor_SMD:R_0603_1608Metric, F.Cu at (70.1, 5.78)
- added R152: 10k, Resistor_SMD:R_0603_1608Metric, F.Cu at (70.1, 8.29)
- added R153: 4.75k, Resistor_SMD:R_0603_1608Metric, F.Cu at (70.1, 10.8)
- added R16: 100k, Resistor_SMD:R_0603_1608Metric, F.Cu at (13.5, 13.3)
- added R17: 100k, Resistor_SMD:R_0603_1608Metric, F.Cu at (13.5, 15.8)
- added R18: 100k, Resistor_SMD:R_0603_1608Metric, F.Cu at (13.5, 18.3)
- added R19: 10, Resistor_SMD:R_0603_1608Metric, F.Cu at (13.5, 20.8)
- added R2: 100, Resistor_SMD:R_0603_1608Metric, F.Cu at (9.53, 13.3)
- added R20: 4.7M, Resistor_SMD:R_0603_1608Metric, F.Cu at (13.5, 23.3)
- added R21: 220k, Resistor_SMD:R_2512_6332Metric, F.Cu at (44.2, 42.0)
- added R22: 2K2, Resistor_SMD:R_0805_2012Metric_Pad1.20x1.40mm_HandSolder, F.Cu at (34.4, 44.6)
- added R23: 220k, Resistor_SMD:R_2512_6332Metric, F.Cu at (44.2, 46.9)
- added R24: 4.75k, Resistor_SMD:R_0603_1608Metric, F.Cu at (13.5, 25.9)
- added R25: 100k, Resistor_SMD:R_0603_1608Metric, F.Cu at (13.5, 28.4)
- added R26: 100k, Resistor_SMD:R_0603_1608Metric, F.Cu at (13.5, 30.9)
- added R27: 4.75k, Resistor_SMD:R_0603_1608Metric, F.Cu at (17.5, 0.76)
- added R28: 4.75k, Resistor_SMD:R_0603_1608Metric, F.Cu at (17.5, 3.27)
- added R29: 10k, Resistor_SMD:R_0603_1608Metric, F.Cu at (17.5, 5.78)
- added R3: 100, Resistor_SMD:R_0603_1608Metric, F.Cu at (9.53, 15.8)
- added R30: 100, Resistor_SMD:R_0603_1608Metric, F.Cu at (17.5, 8.29)
- added R31: 1.2k, Resistor_SMD:R_0603_1608Metric, F.Cu at (17.5, 10.8)
- added R33: 100, Resistor_SMD:R_0603_1608Metric, F.Cu at (17.5, 13.3)
- added R34: 100k, Resistor_SMD:R_2512_6332Metric, F.Cu at (44.2, 51.8)
- added R35: 100, Resistor_SMD:R_0603_1608Metric, F.Cu at (17.5, 15.8)
- added R36: 100, Resistor_SMD:R_0603_1608Metric, F.Cu at (17.5, 18.3)
- added R37: 100, Resistor_SMD:R_0603_1608Metric, F.Cu at (17.5, 20.8)
- added R38: 100, Resistor_SMD:R_0603_1608Metric, F.Cu at (17.5, 23.3)
- added R39: 100, Resistor_SMD:R_0603_1608Metric, F.Cu at (17.5, 25.9)
- added R4: 100, Resistor_SMD:R_0603_1608Metric, F.Cu at (9.53, 18.3)
- added R40: 1, Resistor_SMD:R_0603_1608Metric, F.Cu at (17.5, 28.4)
- added R41: 4.7M, Resistor_SMD:R_0603_1608Metric, F.Cu at (17.5, 30.9)
- added R42: 4.7M, Resistor_SMD:R_0603_1608Metric, F.Cu at (21.6, 0.76)
- added R43: 1, Resistor_SMD:R_0603_1608Metric, F.Cu at (21.6, 3.27)
- added R44: 1, Resistor_SMD:R_0603_1608Metric, F.Cu at (21.6, 5.78)
- added R45: 130k, Resistor_SMD:R_0603_1608Metric, F.Cu at (21.6, 8.29)
- added R46: 1.2k, Resistor_SMD:R_0603_1608Metric, F.Cu at (21.6, 10.8)
- added R47: 806, Resistor_SMD:R_0603_1608Metric, F.Cu at (21.6, 13.3)
- added R48: 0, Resistor_SMD:R_0603_1608Metric, F.Cu at (21.6, 15.8)
- added R49: 1M, Resistor_SMD:R_0603_1608Metric, F.Cu at (21.6, 18.3)
- added R50: 0, Resistor_SMD:R_0603_1608Metric, F.Cu at (21.6, 20.8)
- added R51: 100k, Resistor_SMD:R_0603_1608Metric, F.Cu at (21.6, 23.3)
- added R52: 100k, Resistor_SMD:R_0603_1608Metric, F.Cu at (21.6, 25.9)
- added R53: 100k, Resistor_SMD:R_0603_1608Metric, F.Cu at (21.6, 28.4)
- added R54: 100k, Resistor_SMD:R_0603_1608Metric, F.Cu at (21.6, 30.9)
- added R55: 10k, Resistor_SMD:R_0603_1608Metric, F.Cu at (25.6, 0.76)
- added R56: 10k, Resistor_SMD:R_0603_1608Metric, F.Cu at (25.6, 3.27)
- added R57: 100, Resistor_SMD:R_0603_1608Metric, F.Cu at (25.6, 5.78)
- added R58: 1M, Resistor_SMD:R_0603_1608Metric, F.Cu at (25.6, 8.29)
- added R59: 100k, Resistor_SMD:R_0603_1608Metric, F.Cu at (25.6, 10.8)
- added R6: 1.2k, Resistor_SMD:R_0603_1608Metric, F.Cu at (9.53, 20.8)
- added R60: 1.2k, Resistor_SMD:R_0603_1608Metric, F.Cu at (25.6, 13.3)
- added R61: 10k, Resistor_SMD:R_0603_1608Metric, F.Cu at (25.6, 15.8)
- added R62: 470, Resistor_SMD:R_0603_1608Metric, F.Cu at (25.6, 18.3)
- added R63: 470, Resistor_SMD:R_0603_1608Metric, F.Cu at (25.6, 20.8)
- added R64: 470, Resistor_SMD:R_0603_1608Metric, F.Cu at (25.6, 23.3)
- added R65: 1.5k, Resistor_SMD:R_0603_1608Metric, F.Cu at (25.6, 25.9)
- added R66: 100, Resistor_SMD:R_0603_1608Metric, F.Cu at (56.1, 93.8)
- added R67: 1.2k, Resistor_SMD:R_0603_1608Metric, F.Cu at (56.1, 96.3)
- added R68: 3.9, Resistor_SMD:R_2512_6332Metric, F.Cu at (58.5, 87.6)
- added R69: 100, Resistor_SMD:R_0603_1608Metric, F.Cu at (34.3, 64.9)
- added R7: 806, Resistor_SMD:R_0603_1608Metric, F.Cu at (9.53, 23.3)
- added R70: 1.2k, Resistor_SMD:R_0603_1608Metric, F.Cu at (34.3, 67.4)
- added R71: 3.9, Resistor_SMD:R_2512_6332Metric, F.Cu at (36.6, 58.7)
- added R72: 100, Resistor_SMD:R_0603_1608Metric, F.Cu at (77.9, 79.4)
- added R73: 1.2k, Resistor_SMD:R_0603_1608Metric, F.Cu at (77.9, 81.9)
- added R74: 3.9, Resistor_SMD:R_2512_6332Metric, F.Cu at (80.3, 73.1)
- added R75: 100, Resistor_SMD:R_0603_1608Metric, F.Cu at (23.3, 64.9)
- added R76: 1.2k, Resistor_SMD:R_0603_1608Metric, F.Cu at (23.3, 67.4)
- added R77: 3.9, Resistor_SMD:R_2512_6332Metric, F.Cu at (25.7, 58.7)
- added R78: 100, Resistor_SMD:R_0603_1608Metric, F.Cu at (69.0, 37.2)
- added R79: 1.2k, Resistor_SMD:R_0603_1608Metric, F.Cu at (69.0, 39.7)
- added R8: 10, Resistor_SMD:R_0603_1608Metric, F.Cu at (9.53, 25.9)
- added R80: 3.9, Resistor_SMD:R_2512_6332Metric, F.Cu at (71.4, 31.0)
- added R81: 100, Resistor_SMD:R_0603_1608Metric, F.Cu at (67.0, 64.9)
- added R82: 1.2k, Resistor_SMD:R_0603_1608Metric, F.Cu at (67.0, 67.4)
- added R83: 3.9, Resistor_SMD:R_2512_6332Metric, F.Cu at (69.4, 58.7)
- added R84: 100, Resistor_SMD:R_0603_1608Metric, F.Cu at (67.0, 79.4)
- added R85: 1.2k, Resistor_SMD:R_0603_1608Metric, F.Cu at (67.0, 81.9)
- added R86: 3.9, Resistor_SMD:R_2512_6332Metric, F.Cu at (69.4, 73.1)
- added R87: 100, Resistor_SMD:R_0603_1608Metric, F.Cu at (12.4, 79.4)
- added R88: 1.2k, Resistor_SMD:R_0603_1608Metric, F.Cu at (12.4, 81.9)
- added R89: 3.9, Resistor_SMD:R_2512_6332Metric, F.Cu at (14.8, 73.1)
- added R9: 4.7M, Resistor_SMD:R_0603_1608Metric, F.Cu at (9.53, 28.4)
- added R90: 100, Resistor_SMD:R_0603_1608Metric, F.Cu at (12.4, 64.9)
- added R91: 1.2k, Resistor_SMD:R_0603_1608Metric, F.Cu at (12.4, 67.4)
- added R92: 3.9, Resistor_SMD:R_2512_6332Metric, F.Cu at (14.8, 58.7)
- added R93: 100, Resistor_SMD:R_0603_1608Metric, F.Cu at (45.2, 93.8)
- added R94: 1.2k, Resistor_SMD:R_0603_1608Metric, F.Cu at (45.2, 96.3)
- added R95: 3.9, Resistor_SMD:R_2512_6332Metric, F.Cu at (47.5, 87.6)
- added R96: 100, Resistor_SMD:R_0603_1608Metric, F.Cu at (12.4, 93.8)
- added R97: 1.2k, Resistor_SMD:R_0603_1608Metric, F.Cu at (12.4, 96.3)
- added R98: 3.9, Resistor_SMD:R_2512_6332Metric, F.Cu at (14.8, 87.6)
- added R99: 100, Resistor_SMD:R_0603_1608Metric, F.Cu at (1.50, 79.4)
- added TH1: 100k, Resistor_SMD:R_0805_2012Metric, F.Cu at (29.8, 44.6)
- added TH2: Thermistor_NTC 100k, Resistor_SMD:R_0805_2012Metric, F.Cu at (29.8, 47.6)
- added TH3: 100k, Resistor_SMD:R_0805_2012Metric, F.Cu at (29.8, 50.5)
Routing:
- net /BATT-: vias 0 -> 4
- net /BATT+: vias 0 -> 4
- added copper zone on F.Cu, net /BATT+
- added copper zone on F.Cu, net /BATT-
- removed copper zone on F.Cu, net (none)
Other:
- board text added: "Negative Battery Contact"
- board text added: "Positive Battery Contact"
