File: engineering/electronics/pcbs/BMSJ/kicad/MCU.kicad_sch (KiCad schematic)
At the start: 49 parts, among them J12 CAN, J14 SERIAL, J17 DEBUG, J24 USB, J3 OLED, Q17 BSS138, Q27 BSS138, U17 STM32L476RGT6, U2 HM2108NL, U2 LTC6820, U3 ISO1050DUBR, U4 SFH617A-2X017T, U6 CP2104, Y1 8MHz

Commit message: KiCad_Update
Parts:
- renumbered C6 to C67, C7 to C68, C20 to C69, C8 to C70, C50 to C71, C51 to C72, C52 to C73, C53 to C74, C54 to C75, C84 to C76, C76 to C77, C77 to C78, C78 to C79, C43 to C80, C44 to C81, C45 to C82, C46 to C83, D24 to D45, D25 to D46, J12 to J36, J17 to J37, J24 to J38, J3 to J39, J14 to J40, Q27 to Q35, Q17 to Q36, R6 to R138, R7 to R139, R5 to R140, R36 to R141, R37 to R142, R79 to R143, R170 to R144, R80 to R145, R168 to R146, R81 to R147, R85 to R148, R86 to R149, R82 to R150, R83 to R151, R84 to R152, R87 to R153, U17 to U10, U4 to U11, U6 to U12, U2 to U7, U2 to U8, U3 to U9
