File: engineering/electronics/pcbs/BMSJ/kicad/cell.kicad_sch (KiCad schematic)
At the start: 6 parts, among them Q13 DMG2305UX-7

Commit message: KiCad_Update
Parts:
- renumbered C24 to C43, D12 to D21, Q13 to Q11, R46 to R66, R47 to R67, R45 to R68
