File: engineering/electronics/pcbs/BMSJ/kicad/cell2.kicad_sch (KiCad schematic)
At the start: 6 parts, among them Q3 DMG2305UX-7

Commit message: KiCad_Update
Parts:
- removed C30: 100n, Capacitor_SMD:C_0603_1608Metric, symbol Device:C
- removed D5: PDZ7.5B, Diode_SMD:D_SOD-323, symbol Device:D_Zener
- removed R27: 100, Resistor_SMD:R_0603_1608Metric, symbol Device:R
- added C55: 100n, Capacitor_SMD:C_0603_1608Metric, symbol Device:C
- added D33: PDZ7.5B, Diode_SMD:D_SOD-323, symbol Device:D_Zener
- added R102: 100, Resistor_SMD:R_0603_1608Metric, symbol Device:R
- renumbered Q3 to Q23, R28 to R103, R29 to R104
Connections:
- net C: now also C55.1, D33.1 (K), R102.1
- net C+: now also R102.2
- net CM: now also D33.2 (A)
- net GND2: now also C55.2
