File: engineering/electronics/pcbs/BMSZ/kicad/BMSZ.kicad_pcb (KiCad board)
At the start: 2 copper layers, 0 parts

Commit message: Replace BMSZ with SL_PCB basic layout
Parts:
- added J35: ET60S-D06-0-00-D06-X-V1-S, BMSZ:SAMTEC_ET60S-D06-0-00-D06-X-V1-S, F.Cu at (200.2, 117.6)
Routing:
- net /BATT-: vias 0 -> 4
- net /BATT+: vias 0 -> 4
- added copper zone on F.Cu, net /BATT+
- added copper zone on F.Cu, net /BATT-
Other:
- board outline added: 200 x 115 mm
- board text added: "Negative Battery Contact"
- board text added: "Positive Battery Contact"
